Commit message: ver_0717_第六章完成

File: demo05_ws/src/urdf01_rviz/urdf/xacro/demo02_field.urdf.xacro (robot description, xacro)
@@ -1,7 +1,9 @@
-<robot name="mycar" xmlns:xacro="http://wiki.ros.org/xacro">
+<robot name="mycar"
+    xmlns:xacro="http://wiki.ros.org/xacro">
     <!-- 1.属性定义 -->
     <xacro:property name="PI" value="3.1415926" />
     <xacro:property name="radius" value="0.03" />
     <!-- 2.属性调用 -->
+    <!-- myUsePropertyxxx为随意调用的标签 -->
     <myUsePropertyxxx name="${PI}" />
     <myUsePropertyxxx name="${radius}" />

File: demo05_ws/src/urdf01_rviz/urdf/xacro/demo03_macro.urdf.xacro (robot description, xacro)
@@ -1,5 +1,7 @@
-<robot name="mycar" xmlns:xacro="http://wiki.ros.org/xacro">
+<robot name="mycar"
+    xmlns:xacro="http://wiki.ros.org/xacro">
     <!-- 1.宏定义 -->
     <xacro:macro name="getSum" params="num1 num2">
+        <!-- result为自定义结果标签 -->
         <result value="${num1 + num2}" />
     </xacro:macro>

File: demo05_ws/src/urdf01_rviz/urdf/xacro/demo04_sum.urdf.xacro (robot description, xacro)
@@ -1,3 +1,4 @@
-<robot name="mycar" xmlns:xacro="http://wiki.ros.org/xacro">
+<robot name="mycar"
+    xmlns:xacro="http://wiki.ros.org/xacro">
     <!-- 演示文件包含 -->
     <xacro:include filename="demo02_field.urdf.xacro" />

File: demo05_ws/src/urdf01_rviz/urdf/xacro/demo05_car_base.urdf (robot description, URDF)
Before this commit: robot mycar, 2 links, 1 joints
Links:
- added link back_wheel; visual sphere radius=0.0075
- added link front_wheel; visual sphere radius=0.0075
- added link left_wheel; visual cylinder length=0.015 radius=0.0325
- added link right_wheel; visual cylinder length=0.015 radius=0.0325
Joints:
- added joint back2link: type continuous, parent base_link, child back_wheel, origin xyz=-0.08 0 -0.0475 rpy=0 0 0, axis 0 1 0
- added joint front2link: type continuous, parent base_link, child front_wheel, origin xyz=0.08 0 -0.0475 rpy=0 0 0, axis 0 1 0
- added joint left2link: type continuous, parent base_link, child left_wheel, origin xyz=0 0.1 -0.0225 rpy=0 0 0, axis 0 1 0
- added joint right2link: type continuous, parent base_link, child right_wheel, origin xyz=0 -0.1 -0.0225 rpy=0 0 0, axis 0 1 0

File: demo05_ws/src/urdf01_rviz/urdf/xacro/demo05_car_base.urdf.xacro (robot description, xacro)
@@ -1,3 +1,4 @@
-<robot name="mycar" xmlns:xacro="http://wiki.ros.org/xacro">
+<robot name="mycar"
+    xmlns:xacro="http://wiki.ros.org/xacro">
     <xacro:property name="footprint_radius" value="0.001" />
     <!-- 1.添加base_footprint -->
@@ -33,8 +34,12 @@
         <origin xyz="0 0 0.055" rpy="0 0 0" />
     </joint>
-    <xacro:property name="wheel_radius" value="0.0325" /><!-- 半径 -->
-    <xacro:property name="wheel_length" value="0.015" /><!-- 宽度 -->
-    <xacro:property name="PI" value="3.1415926" /><!-- 宽度 -->
-    <xacro:property name="wheel_joint_z" value="${-(base_length/2 + lidi - wheel_radius)}" /><!-- 宽度 -->
+    <xacro:property name="wheel_radius" value="0.0325" />
+    <!-- 半径 -->
+    <xacro:property name="wheel_length" value="0.015" />
+    <!-- 宽度 -->
+    <xacro:property name="PI" value="3.1415926" />
+    <!-- PI -->
+    <xacro:property name="wheel_joint_z" value="${-(base_length/2 + lidi - wheel_radius)}" />
+    <!-- z偏移量 -->
     <!--
         wheel_name: left or right
@@ -42,5 +47,5 @@
      -->
     <xacro:macro name="wheel_func" params="wheel_name flag">
-    <!-- 3.驱动轮  -->
+        <!-- 3.驱动轮  -->
         <link name="${wheel_name}_wheel">
             <visual>
@@ -57,11 +62,16 @@
             <parent link="base_link" />
             <child link="${wheel_name}_wheel" />
-            <!-- z=0.055-0.0325 -->
+            <!--
+                x 无偏移
+                y 车体半径
+                z z = 车体高度/2 + 离地间距 - 车轮半径
+             -->
             <origin xyz="0 ${0.1 * flag} ${wheel_joint_z}" rpy="0 0 0" />
             <axis xyz="0 1 0" />
         </joint>
     </xacro:macro>
-    <xacro:property name="small_wheel_radius" value="0.0075" /><!-- 半径 -->
-    <!-- z的偏移量=车体高度/2 + 离地间距 - 万向轮半价 -->
+    <xacro:property name="small_wheel_radius" value="0.0075" />
+    <!-- 半径 -->
+    <!-- z的偏移量 = 车体高度/2 + 离地间距 - 万向轮半径 -->
     <xacro:property name="small_joint_z" value="${-(base_length/2 + lidi - small_wheel_radius)}" />
     <xacro:macro name="small_wheel_func" params="small_wheel_name flag">

File: demo05_ws/src/urdf01_rviz/urdf/xacro/demo06_car_camera.urdf.xacro (robot description, xacro)
@@ -1,11 +1,19 @@
 <!-- 摄像头相关的 xacro 文件 -->
-<robot name="my_camera" xmlns:xacro="http://wiki.ros.org/xacro">
+<robot name="my_camera"
+    xmlns:xacro="http://wiki.ros.org/xacro">
     <!-- 摄像头属性 -->
-    <xacro:property name="camera_length" value="0.01" /> <!-- 摄像头长度(x) -->
-    <xacro:property name="camera_width" value="0.025" /> <!-- 摄像头宽度(y) -->
-    <xacro:property name="camera_height" value="0.025" /> <!-- 摄像头高度(z) -->
-    <xacro:property name="camera_x" value="0.08" /> <!-- 摄像头安装的x坐标 -->
-    <xacro:property name="camera_y" value="0.0" /> <!-- 摄像头安装的y坐标 -->
-    <xacro:property name="camera_z" value="${base_length / 2 + camera_height / 2}" /> <!-- 摄像头安装的z坐标:底盘高度 / 2 + 摄像头高度 / 2  -->
+    <xacro:property name="camera_length" value="0.01" />
+    <!-- 摄像头长度(x) -->
+    <xacro:property name="camera_width" value="0.025" />
+    <!-- 摄像头宽度(y) -->
+    <xacro:property name="camera_height" value="0.025" />
+    <!-- 摄像头高度(z) -->
+    <xacro:property name="camera_x" value="0.08" />
+    <!-- 摄像头安装的x坐标 -->
+    <xacro:property name="camera_y" value="0.0" />
+    <!-- 摄像头安装的y坐标 -->
+    <!-- 这里的base_length在demo05_car_base.urdf.xacro已经定义过，使用时需要先include demo05_car_base.urdf.xacro -->
+    <xacro:property name="camera_z" value="${base_length / 2 + camera_height / 2}" />
+    <!-- 摄像头安装的z坐标:底盘高度 / 2 + 摄像头高度 / 2  -->
     <!-- 摄像头关节以及link -->
     <link name="camera">
@@ -15,5 +23,5 @@
             </geometry>
             <origin xyz="0.0 0.0 0.0" rpy="0.0 0.0 0.0" />
-            <material name="black" >
+            <material name="black">
                 <color rgba="0 0 0 0.8" />
             </material>

File: demo05_ws/src/urdf01_rviz/urdf/xacro/demo07_car_laser.urdf.xacro (robot description, xacro)
@@ -2,11 +2,17 @@
     小车底盘添加雷达
 -->
-<robot name="my_laser" xmlns:xacro="http://wiki.ros.org/xacro">
+<robot name="my_laser"
+    xmlns:xacro="http://wiki.ros.org/xacro">
     <!-- 雷达支架 -->
-    <xacro:property name="support_length" value="0.05" /> <!-- 支架长度 -->
-    <xacro:property name="support_radius" value="0.01" /> <!-- 支架半径 -->
-    <xacro:property name="support_x" value="0.0" /> <!-- 支架安装的x坐标 -->
-    <xacro:property name="support_y" value="0.0" /> <!-- 支架安装的y坐标 -->
-    <xacro:property name="support_z" value="${base_length / 2 + support_length / 2}" /> <!-- 支架安装的z坐标:底盘高度 / 2 + 支架高度 / 2  -->
+    <xacro:property name="support_length" value="0.05" />
+    <!-- 支架长度 -->
+    <xacro:property name="support_radius" value="0.01" />
+    <!-- 支架半径 -->
+    <xacro:property name="support_x" value="0.0" />
+    <!-- 支架安装的x坐标 -->
+    <xacro:property name="support_y" value="0.0" />
+    <!-- 支架安装的y坐标 -->
+    <xacro:property name="support_z" value="${base_length / 2 + support_length / 2}" />
+    <!-- 支架安装的z坐标:底盘高度 / 2 + 支架高度 / 2  -->
     <link name="support">
         <visual>
@@ -26,9 +32,14 @@
     </joint>
     <!-- 雷达属性 -->
-    <xacro:property name="laser_length" value="0.05" /> <!-- 雷达长度 -->
-    <xacro:property name="laser_radius" value="0.03" /> <!-- 雷达半径 -->
-    <xacro:property name="laser_x" value="0.0" /> <!-- 雷达安装的x坐标 -->
-    <xacro:property name="laser_y" value="0.0" /> <!-- 雷达安装的y坐标 -->
-    <xacro:property name="laser_z" value="${support_length / 2 + laser_length / 2}" /> <!-- 雷达安装的z坐标:支架高度 / 2 + 雷达高度 / 2  -->
+    <xacro:property name="laser_length" value="0.05" />
+    <!-- 雷达长度 -->
+    <xacro:property name="laser_radius" value="0.03" />
+    <!-- 雷达半径 -->
+    <xacro:property name="laser_x" value="0.0" />
+    <!-- 雷达安装的x坐标 -->
+    <xacro:property name="laser_y" value="0.0" />
+    <!-- 雷达安装的y坐标 -->
+    <xacro:property name="laser_z" value="${support_length / 2 + laser_length / 2}" />
+    <!-- 雷达安装的z坐标:支架高度 / 2 + 雷达高度 / 2  -->
     <!-- 雷达关节以及link -->
     <link name="laser">
@@ -38,5 +49,5 @@
             </geometry>
             <origin xyz="0.0 0.0 0.0" rpy="0.0 0.0 0.0" />
-            <material name="black" >
+            <material name="black">
                 <color rgba="0 0 0 0.8" />
             </material>

File: demo05_ws/src/urdf01_rviz/urdf/xacro/demo08_car.urdf.xacro (robot description, xacro)
@@ -1,3 +1,4 @@
-<robot name="mycar" xmlns:xacro="http://wiki.ros.org/xacro">
+<robot name="mycar"
+    xmlns:xacro="http://wiki.ros.org/xacro">
     <!-- 包含底盘，摄像头与雷达的xacro文件  -->
     <xacro:include filename="demo05_car_base.urdf.xacro"/>

File: demo05_ws/src/urdf02_gazebo/urdf/demo06_car_camera.urdf.xacro (robot description, xacro)
@@ -1,11 +1,20 @@
 <!-- 摄像头相关的 xacro 文件 -->
-<robot name="my_camera" xmlns:xacro="http://wiki.ros.org/xacro">
+<robot name="my_camera"
+    xmlns:xacro="http://wiki.ros.org/xacro">
     <!-- 摄像头属性 -->
-    <xacro:property name="camera_length" value="0.01" /> <!-- 摄像头长度(x) -->
-    <xacro:property name="camera_width" value="0.025" /> <!-- 摄像头宽度(y) -->
-    <xacro:property name="camera_height" value="0.025" /> <!-- 摄像头高度(z) -->
-    <xacro:property name="camera_x" value="0.08" /> <!-- 摄像头安装的x坐标 -->
-    <xacro:property name="camera_y" value="0.0" /> <!-- 摄像头安装的y坐标 -->
-    <xacro:property name="camera_z" value="${base_length / 2 + camera_height / 2}" /> <!-- 摄像头安装的z坐标:底盘高度 / 2 + 摄像头高度 / 2  -->
+    <!-- 摄像头质量 -->
+    <xacro:property name="camera_mass" value="0.01" />
+    <!-- 摄像头长度(x) -->
+    <xacro:property name="camera_length" value="0.01" />
+    <!-- 摄像头宽度(y) -->
+    <xacro:property name="camera_width" value="0.025" />
+    <!-- 摄像头高度(z) -->
+    <xacro:property name="camera_height" value="0.025" />
+    <!-- 摄像头安装的x坐标 -->
+    <xacro:property name="camera_x" value="0.08" />
+    <!-- 摄像头安装的y坐标 -->
+    <xacro:property name="camera_y" value="0.0" />
+    <!-- 摄像头安装的z坐标:底盘高度 / 2 + 摄像头高度 / 2  -->
+    <xacro:property name="camera_z" value="${base_length / 2 + camera_height / 2}" />
     <!-- 摄像头关节以及link -->
     <link name="camera">
@@ -15,8 +24,15 @@
             </geometry>
             <origin xyz="0.0 0.0 0.0" rpy="0.0 0.0 0.0" />
-            <material name="black" >
+            <material name="black">
                 <color rgba="0 0 0 0.8" />
             </material>
         </visual>
+        <collision>
+            <geometry>
+                <box size="${camera_length} ${camera_width} ${camera_height}" />
+            </geometry>
+            <origin xyz="0.0 0.0 0.0" rpy="0.0 0.0 0.0" />
+        </collision>
+        <xacro:Box_inertial_matrix m="${camera_mass}" l="${camera_length}" w="${camera_width}" h="${camera_height}" />
     </link>
     <gazebo reference="camera">

File: demo05_ws/src/urdf02_gazebo/urdf/demo07_car_laser.urdf.xacro (robot description, xacro)
@@ -2,11 +2,19 @@
     小车底盘添加雷达
 -->
-<robot name="my_laser" xmlns:xacro="http://wiki.ros.org/xacro">
+<robot name="my_laser"
+    xmlns:xacro="http://wiki.ros.org/xacro">
     <!-- 雷达支架 -->
-    <xacro:property name="support_length" value="0.05" /> <!-- 支架长度 -->
-    <xacro:property name="support_radius" value="0.01" /> <!-- 支架半径 -->
-    <xacro:property name="support_x" value="0.0" /> <!-- 支架安装的x坐标 -->
-    <xacro:property name="support_y" value="0.0" /> <!-- 支架安装的y坐标 -->
-    <xacro:property name="support_z" value="${base_length / 2 + support_length / 2}" /> <!-- 支架安装的z坐标:底盘高度 / 2 + 支架高度 / 2  -->
+    <!-- 支架质量 -->
+    <xacro:property name="support_mass" value="0.1" />
+    <!-- 支架长度 -->
+    <xacro:property name="support_length" value="0.05" />
+    <!-- 支架半径 -->
+    <xacro:property name="support_radius" value="0.01" />
+    <!-- 支架安装的x坐标 -->
+    <xacro:property name="support_x" value="0.0" />
+    <!-- 支架安装的y坐标 -->
+    <xacro:property name="support_y" value="0.0" />
+    <!-- 支架安装的z坐标:底盘高度 / 2 + 支架高度 / 2  -->
+    <xacro:property name="support_z" value="${base_length / 2 + support_length / 2}" />
     <link name="support">
         <visual>
@@ -19,4 +27,11 @@
             </material>
         </visual>
+        <collision>
+            <geometry>
+                <cylinder radius="${support_radius}" length="${support_length}" />
+            </geometry>
+            <origin xyz="0.0 0.0 0.0" rpy="0.0 0.0 0.0" />
+        </collision>
+        <xacro:cylinder_inertial_matrix m="${support_mass}" r="${support_radius}" h="${support_length}" />
     </link>
     <gazebo reference="support">
@@ -29,9 +44,16 @@
     </joint>
     <!-- 雷达属性 -->
-    <xacro:property name="laser_length" value="0.05" /> <!-- 雷达长度 -->
-    <xacro:property name="laser_radius" value="0.03" /> <!-- 雷达半径 -->
-    <xacro:property name="laser_x" value="0.0" /> <!-- 雷达安装的x坐标 -->
-    <xacro:property name="laser_y" value="0.0" /> <!-- 雷达安装的y坐标 -->
-    <xacro:property name="laser_z" value="${support_length / 2 + laser_length / 2}" /> <!-- 雷达安装的z坐标:支架高度 / 2 + 雷达高度 / 2  -->
+    <!-- 雷达质量 -->
+    <xacro:property name="laser_mass" value="0.01" />
+    <!-- 雷达长度 -->
+    <xacro:property name="laser_length" value="0.05" />
+    <!-- 雷达半径 -->
+    <xacro:property name="laser_radius" value="0.03" />
+    <!-- 雷达安装的x坐标 -->
+    <xacro:property name="laser_x" value="0.0" />
+    <!-- 雷达安装的y坐标 -->
+    <xacro:property name="laser_y" value="0.0" />
+    <!-- 雷达安装的z坐标:支架高度 / 2 + 雷达高度 / 2  -->
+    <xacro:property name="laser_z" value="${support_length / 2 + laser_length / 2}" />
     <!-- 雷达关节以及link -->
     <link name="laser">
@@ -41,9 +63,19 @@
             </geometry>
             <origin xyz="0.0 0.0 0.0" rpy="0.0 0.0 0.0" />
-            <material name="black" >
+            <material name="black">
                 <color rgba="0 0 0 0.8" />
             </material>
         </visual>
+        <collision>
+            <geometry>
+                <cylinder radius="${laser_radius}" length="${laser_length}" />
+            </geometry>
+            <origin xyz="0.0 0.0 0.0" rpy="0.0 0.0 0.0" />
+        </collision>
+        <xacro:cylinder_inertial_matrix m="${laser_mass}" r="${laser_radius}" h="${laser_length}" />
     </link>
+    <gazebo reference="laser">
+        <material>Gazebo/Red</material>
+    </gazebo>
     <joint name="laser2support" type="fixed">
         <parent link="support" />

File: demo05_ws/src/urdf02_gazebo/urdf/demo08_car.urdf.xacro (robot description, xacro)
@@ -1,3 +1,4 @@
-<robot name="mycar" xmlns:xacro="http://wiki.ros.org/xacro">
+<robot name="mycar"
+    xmlns:xacro="http://wiki.ros.org/xacro">
     <!-- 包含惯性矩阵文件 -->
     <xacro:include filename="head.xacro"/>

File: demo05_ws/src/urdf02_gazebo/urdf/gazebo/camera.xacro (robot description, xacro)
@@ -1,8 +1,9 @@
-<robot name="my_sensors" xmlns:xacro="http://wiki.ros.org/xacro">
-  <!-- 被引用的link -->
+<robot name="my_sensors"
+  xmlns:xacro="http://wiki.ros.org/xacro">
+  <!-- 被引用的link名字，这里link名就叫camera -->
   <gazebo reference="camera">
     <!-- 类型设置为 camara -->
     <sensor type="camera" name="camera_node">
-      <update_rate>30.0</update_rate> <!-- 更新频率 -->
+      <update_rate>30.0</update_rate>      <!-- 更新频率 -->
       <!-- 摄像头基本信息设置 -->
       <camera name="head">
@@ -27,7 +28,9 @@
         <alwaysOn>true</alwaysOn>
         <updateRate>0.0</updateRate>
+        <!-- 为发布话题设置的命名空间 随意设置 -->
         <cameraName>/camera</cameraName>
         <imageTopicName>image_raw</imageTopicName>
         <cameraInfoTopicName>camera_info</cameraInfoTopicName>
+        <!-- 被引用的link名字，这里link名就叫camera -->
         <frameName>camera</frameName>
         <hackBaseline>0.07</hackBaseline>

File: demo05_ws/src/urdf02_gazebo/urdf/gazebo/kinect.xacro (robot description, xacro)
@@ -1,38 +1,40 @@
-<robot name="my_sensors" xmlns:xacro="http://wiki.ros.org/xacro">
-    <gazebo reference="support">
-      <sensor type="depth" name="camera">
-        <always_on>true</always_on>
-        <update_rate>20.0</update_rate>
-        <camera>
-          <horizontal_fov>${60.0*PI/180.0}</horizontal_fov>
-          <image>
-            <format>R8G8B8</format>
-            <width>640</width>
-            <height>480</height>
-          </image>
-          <clip>
-            <near>0.05</near>
-            <far>8.0</far>
-          </clip>
-        </camera>
-        <plugin name="kinect_camera_controller" filename="libgazebo_ros_openni_kinect.so">
-          <cameraName>camera</cameraName>
-          <alwaysOn>true</alwaysOn>
-          <updateRate>10</updateRate>
-          <imageTopicName>rgb/image_raw</imageTopicName>
-          <depthImageTopicName>depth/image_raw</depthImageTopicName>
-          <pointCloudTopicName>depth/points</pointCloudTopicName>
-          <cameraInfoTopicName>rgb/camera_info</cameraInfoTopicName>
-          <depthImageCameraInfoTopicName>depth/camera_info</depthImageCameraInfoTopicName>
-          <frameName>support_depth</frameName>
-          <baseline>0.1</baseline>
-          <distortion_k1>0.0</distortion_k1>
-          <distortion_k2>0.0</distortion_k2>
-          <distortion_k3>0.0</distortion_k3>
-          <distortion_t1>0.0</distortion_t1>
-          <distortion_t2>0.0</distortion_t2>
-          <pointCloudCutoff>0.4</pointCloudCutoff>
-        </plugin>
-      </sensor>
-    </gazebo>
+<robot name="my_sensors"
+  xmlns:xacro="http://wiki.ros.org/xacro">
+  <gazebo reference="support">
+    <sensor type="depth" name="camera">
+      <always_on>true</always_on>
+      <update_rate>20.0</update_rate>
+      <camera>
+        <horizontal_fov>${60.0*PI/180.0}</horizontal_fov>
+        <image>
+          <format>R8G8B8</format>
+          <width>640</width>
+          <height>480</height>
+        </image>
+        <clip>
+          <near>0.05</near>
+          <far>8.0</far>
+        </clip>
+      </camera>
+      <plugin name="kinect_camera_controller" filename="libgazebo_ros_openni_kinect.so">
+        <!-- 命名空间 -->
+        <cameraName>/camera_depth</cameraName>
+        <alwaysOn>true</alwaysOn>
+        <updateRate>10</updateRate>
+        <imageTopicName>rgb/image_raw</imageTopicName>
+        <depthImageTopicName>depth/image_raw</depthImageTopicName>
+        <pointCloudTopicName>depth/points</pointCloudTopicName>
+        <cameraInfoTopicName>rgb/camera_info</cameraInfoTopicName>
+        <depthImageCameraInfoTopicName>depth/camera_info</depthImageCameraInfoTopicName>
+        <frameName>support_depth</frameName>
+        <baseline>0.1</baseline>
+        <distortion_k1>0.0</distortion_k1>
+        <distortion_k2>0.0</distortion_k2>
+        <distortion_k3>0.0</distortion_k3>
+        <distortion_t1>0.0</distortion_t1>
+        <distortion_t2>0.0</distortion_t2>
+        <pointCloudCutoff>0.4</pointCloudCutoff>
+      </plugin>
+    </sensor>
+  </gazebo>
 </robot>

File: demo05_ws/src/urdf02_gazebo/urdf/gazebo/laser.xacro (robot description, xacro)
@@ -1,14 +1,19 @@
-<robot name="my_sensors" xmlns:xacro="http://wiki.ros.org/xacro">
+<robot name="my_sensors"
+  xmlns:xacro="http://wiki.ros.org/xacro">
   <!-- 雷达 -->
+  <!-- 这里的"laser"是xacro里雷达连杆的名称 -->
   <gazebo reference="laser">
     <sensor type="ray" name="rplidar">
       <pose>0 0 0 0 0 0</pose>
       <visualize>true</visualize>
-      <update_rate>20</update_rate>
+      <update_rate>5</update_rate>
       <ray>
         <scan>
           <horizontal>
+            <!-- 旋转一圈多少射线 -->
             <samples>360</samples>
+            <!-- 测距的射线间隔：ex. 设成10表示每10个射线测距1次 -->
             <resolution>1</resolution>
+            <!-- 雷达测量范围：-3rad——3rad圆周范围 -->
             <min_angle>-3</min_angle>
             <max_angle>3</max_angle>
@@ -16,9 +21,12 @@
         </scan>
         <range>
+          <!-- 雷达采样距离设置 这里是0.1——5m -->
           <min>0.10</min>
-          <max>30.0</max>
+          <max>5.0</max>
+          <!-- resolution为雷达精度0.01m(1cm) -->
           <resolution>0.01</resolution>
         </range>
         <noise>
+          <!-- 高斯噪声 -->
           <type>gaussian</type>
           <mean>0.0</mean>
@@ -28,4 +36,5 @@
       <plugin name="gazebo_rplidar" filename="libgazebo_ros_laser.so">
         <topicName>/scan</topicName>
+        <!-- 这里的"laser"是xacro里雷达连杆的名称 -->
         <frameName>laser</frameName>
       </plugin>

File: demo05_ws/src/urdf02_gazebo/urdf/gazebo/move.xacro (robot description, xacro)
@@ -1,3 +1,4 @@
-<robot name="my_car_move" xmlns:xacro="http://wiki.ros.org/xacro">
+<robot name="my_car_move"
+    xmlns:xacro="http://wiki.ros.org/xacro">
     <!-- 传动实现:用于连接控制器与关节 -->
     <xacro:macro name="joint_trans" params="joint_name">
@@ -14,5 +15,5 @@
         </transmission>
     </xacro:macro>
-    <!-- 每一个驱动轮都需要配置传动装置 -->
+    <!-- 每一个驱动轮都需要配置传动装置 需要修改此处的joint_name -->
     <xacro:joint_trans joint_name="left2link" />
     <xacro:joint_trans joint_name="right2link" />
@@ -28,15 +29,19 @@
             <updateRate>100.0</updateRate>
             <legacyMode>true</legacyMode>
-            <leftJoint>left2link</leftJoint> <!-- 左轮 -->
-            <rightJoint>right2link</rightJoint> <!-- 右轮 -->
-            <wheelSeparation>${base_radius * 2}</wheelSeparation> <!-- 车轮间距 -->
-            <wheelDiameter>${wheel_radius * 2}</wheelDiameter> <!-- 车轮直径 -->
+            <!-- 需要修改此处的joint_name -->
+            <leftJoint>left2link</leftJoint>            <!-- 左轮 -->
+            <rightJoint>right2link</rightJoint>            <!-- 右轮 -->
+            <!-- 需要修改此处的base_radius -->
+            <wheelSeparation>${base_radius * 2}</wheelSeparation>            <!-- 车轮间距 -->
+            <!-- 需要修改此处的wheel_radius -->
+            <wheelDiameter>${wheel_radius * 2}</wheelDiameter>            <!-- 车轮直径 -->
             <broadcastTF>1</broadcastTF>
             <wheelTorque>30</wheelTorque>
             <wheelAcceleration>1.8</wheelAcceleration>
-            <commandTopic>cmd_vel</commandTopic> <!-- 运动控制话题 -->
+            <commandTopic>cmd_vel</commandTopic>            <!-- 运动控制话题 -->
             <odometryFrame>odom</odometryFrame>
-            <odometryTopic>odom</odometryTopic> <!-- 里程计话题 -->
-            <robotBaseFrame>base_footprint</robotBaseFrame> <!-- 根坐标系 -->
+            <odometryTopic>odom</odometryTopic>            <!-- 里程计话题 -->
+            <!-- 需要修改此处的根坐标系 -->
+            <robotBaseFrame>base_footprint</robotBaseFrame>            <!-- 根坐标系 -->
         </plugin>
     </gazebo>
