Commit message: ver_0722_demo05_car_base.urdf.xacro_修改

File: demo05_ws/src/urdf02_gazebo/urdf/demo05_car_base.urdf.xacro (robot description, xacro)
@@ -1,3 +1,4 @@
-<robot name="mycar" xmlns:xacro="http://wiki.ros.org/xacro">
+<robot name="mycar"
+    xmlns:xacro="http://wiki.ros.org/xacro">
     <xacro:property name="footprint_radius" value="0.001" />
     <!-- 1.添加base_footprint -->
@@ -45,9 +46,14 @@
         <origin xyz="0 0 0.055" rpy="0 0 0" />
     </joint>
-    <xacro:property name="wheel_radius" value="0.0325" /><!-- 半径 -->
-    <xacro:property name="wheel_length" value="0.015" /><!-- 宽度 -->
-    <xacro:property name="wheel_mess" value="0.05" /><!-- 宽度 -->
-    <xacro:property name="PI" value="3.1415926" /><!-- 宽度 -->
-    <xacro:property name="wheel_joint_z" value="${-(base_length/2 + lidi - wheel_radius)}" /><!-- 宽度 -->
+    <xacro:property name="wheel_radius" value="0.0325" />
+    <!-- 半径 -->
+    <xacro:property name="wheel_length" value="0.015" />
+    <!-- 宽度 -->
+    <xacro:property name="wheel_mess" value="0.05" />
+    <!-- 宽度 -->
+    <xacro:property name="PI" value="3.1415926" />
+    <!-- 宽度 -->
+    <xacro:property name="wheel_joint_z" value="${-(base_length/2 + lidi - wheel_radius)}" />
+    <!-- 宽度 -->
     <!--
         wheel_name: left or right
@@ -55,5 +61,5 @@
      -->
     <xacro:macro name="wheel_func" params="wheel_name flag">
-    <!-- 3.驱动轮  -->
+        <!-- 3.驱动轮  -->
         <link name="${wheel_name}_wheel">
             <visual>
@@ -86,6 +92,8 @@
         </joint>
     </xacro:macro>
-    <xacro:property name="small_wheel_radius" value="0.0075" /><!-- 半径 -->
-    <xacro:property name="small_wheel_mess" value="0.01" /><!-- 半径 -->
+    <xacro:property name="small_wheel_radius" value="0.0075" />
+    <!-- 半径 -->
+    <xacro:property name="small_wheel_mess" value="0.01" />
+    <!-- 半径 -->
     <!-- z的偏移量=车体高度/2 + 离地间距 - 万向轮半价 -->
     <xacro:property name="small_joint_z" value="${-(base_length/2 + lidi - small_wheel_radius)}" />
